File: avionics/avionics.kicad_sch (KiCad schematic)
At the start: 6 parts, among them U1 Teensy4.1

Commit message: hw: make board smaller, misc hotfixes
Parts:
- removed TP2: TP_I2C_SCL, TestPoint:TestPoint_Pad_D1.5mm, symbol Connector:TestPoint
- removed TP3: TP_I2C_SDA, TestPoint:TestPoint_Pad_D1.5mm, symbol Connector:TestPoint
- added C1: 100n, Capacitor_SMD:C_0603_1608Metric, symbol Device:C
- added R1, R2, R3: 33, Resistor_SMD:R_0603_1608Metric, symbol Device:R
- added SW1: ~{SW_GUIDANCE_EN}, Button_Switch_THT:SW_PUSH_6mm, symbol Switch:SW_Push
- R4: renamed from R1; footprint Resistor_SMD:R_0805_2012Metric_Pad1.20x1.40mm_HandSolder -> Resistor_SMD:R_0603_1608Metric
- R5: renamed from R2; footprint Resistor_SMD:R_0805_2012Metric_Pad1.20x1.40mm_HandSolder -> Resistor_SMD:R_0603_1608Metric
Connections:
- net GND: now also C1.2, SW1.2
- net IMU/CS_ACC: now also R1.1; no longer U1.12 (10_CS_MQSR)
- net IMU/MISO: now also R3.1; no longer U1.14 (12_MISO_MQSL)
- net IMU/MOSI: now also R2.1; no longer U1.13 (11_MOSI_CTX1)
- net PSU/BAT_CELL_0: now also U1.32 (40_A16); no longer U1.33 (41_A17)
- net PSU/BAT_CELL_1: now also U1.33 (41_A17); no longer U1.32 (40_A16)
- net at U1.22 (30_CRX3): now also C1.1, SW1.1
- new net: R3.2, U1.14 (12_MISO_MQSL)
- new net: R1.2, U1.12 (10_CS_MQSR)
- new net: R2.2, U1.13 (11_MOSI_CTX1)
- no-connect marks 41 -> 40

Commit message: hw: order pcb
Parts:
- added R10, R9: 2.7k, Resistor_SMD:R_0603_1608Metric, symbol Device:R
- added R4, R5, R6: 33, Resistor_SMD:R_0603_1608Metric, symbol Device:R
- C1: DigiKey Part Number (none) -> 399-C0603C104K5RACTUCT-ND; Mouser Part Number (none) -> 603-CC603KRX5R9BB104
- R1, R2, R3: DigiKey Part Number (none) -> 13-RC0603FR-0733RLCT-ND; Mouser Part Number (none) -> 603-RC0603FR-7W33RL
- R7: renamed from R4; DigiKey Part Number (none) -> 311-2.70KHRCT-ND; Mouser Part Number (none) -> 71-CRCW0603-2.7K-E3
- R8: renamed from R5; DigiKey Part Number (none) -> 311-2.70KHRCT-ND; Mouser Part Number (none) -> 71-CRCW0603-2.7K-E3
- SW1: value ~{SW_GUIDANCE_EN} -> 6x6mm Switch
- TP1: now left out of the parts list
- U1: DigiKey Part Number (none) -> 1568-20359-ND
Connections:
- net +3.3V: now also R10.1, R9.1; no longer U1.15 (3V3)
- net SPI_SCK: now also R4.2; no longer U1.35 (13_SCK_LED)
- net SW_GUIDANCE: now reaches C1.1, SW1.1, U1.22 (30_CRX3)
- net I2C_OUT_SCL: now reaches U1.16 (24_A10_TX6_SCL2)
- net I2C_OUT_SCL: now also R9.2
- net I2C_OUT_SDA: now reaches U1.17 (25_A11_RX6_SDA2)
- net I2C_OUT_SDA: now also R10.2
- net at U1.26 (34_RX8): now also R6.1
- net at U1.27 (35_TX8): now also R5.1
- net Barometer/SCL renamed I2C_SCL
- net Barometer/SDA renamed I2C_SDA
- net IMU/CS_ACC renamed SPI_CS
- net IMU/INT_ACC renamed INT_ACC
- net IMU/INT_GYR renamed INT_GYR
- net IMU/MISO renamed SPI_MISO
- net IMU/MOSI renamed SPI_MOSI
- net IMU_CS_GYR: no longer names the net of U1.29 (37_CS)
- net PSU/BAT_CELL_0: no longer names the net of U1.32 (40_A16)
- net PSU/BAT_CELL_1 renamed BAT_VOLTAGE
- net Pyro_and_servos/PYRO_0 renamed PYRO_0
- net Pyro_and_servos/PYRO_0_CONT renamed PYRO_0_CONT
- net Pyro_and_servos/SERVO_0_PWM renamed SERVO_3_PWM
- net Pyro_and_servos/SERVO_1_PWM renamed SERVO_2_PWM
- net Pyro_and_servos/SERVO_2_PWM renamed SERVO_1_PWM
- net Pyro_and_servos/SERVO_3_PWM renamed SERVO_0_PWM
- new net: R4.1, U1.35 (13_SCK_LED)
- new net UART_RX: R6.2
- new net UART_TX: R5.2
- no-connect marks 40 -> 39
Other:
- added sheet Peripheral Connectors (peripherals.kicad_sch)
- sheet IMU ports: added CS; removed CS_ACC, CS_GYR
- sheet PSU ports: added BAT_VOLTAGE; removed BAT_CELL_0, BAT_CELL_1
- moved on the sheet: C1, R1, R2, R3, R7, R8, SW1, TP1
