File: avionics/barometer.kicad_sch (KiCad schematic)
At the start: 3 parts, among them U3 BMP280

Commit message: hw: make board smaller, misc hotfixes
Parts:
- C4: renamed from C3; footprint Capacitor_SMD:C_0805_2012Metric_Pad1.18x1.45mm_HandSolder -> Capacitor_SMD:C_0603_1608Metric
- C5: renamed from C4; footprint Capacitor_SMD:C_0805_2012Metric_Pad1.18x1.45mm_HandSolder -> Capacitor_SMD:C_0603_1608Metric
Changed lines of the file:
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@@
 		(dnp no)
 		(fields_autoplaced yes)
-		(property "Reference" "C4"
+		(property "Reference" "C5"
 			(at 173.99 97.7899 0)
 			(effects
@@
 			)
 		)
-		(property "Footprint" "Capacitor_SMD:C_0805_2012Metric_Pad1.18x1.45mm_HandSolder"
+		(property "Footprint" "Capacitor_SMD:C_0603_1608Metric"
 			(at 171.1452 102.87 0)
 			(effects
@@
 			(project "avionics"
 				(path "/5552e11b-fce5-44fd-aeb8-61bf7d07571f/67ffb272-e6d8-49a0-b0ad-d980ce69be53"
-					(reference "C4")
+					(reference "C5")
 					(unit 1)
 				)
@@
 		(dnp no)
 		(fields_autoplaced yes)
-		(property "Reference" "#PWR012"
+		(property "Reference" "#PWR013"
 			(at 140.97 116.84 0)
 			(effects
@@
 			(project "avionics"
 				(path "/5552e11b-fce5-44fd-aeb8-61bf7d07571f/67ffb272-e6d8-49a0-b0ad-d980ce69be53"
-					(reference "#PWR012")
+					(reference "#PWR013")
 					(unit 1)
 				)
@@
 		(dnp no)
 		(fields_autoplaced yes)
-		(property "Reference" "#PWR011"
+		(property "Reference" "#PWR012"
 			(at 140.97 86.36 0)
 			(effects
@@
 			(project "avionics"
 				(path "/5552e11b-fce5-44fd-aeb8-61bf7d07571f/67ffb272-e6d8-49a0-b0ad-d980ce69be53"
-					(reference "#PWR011")
+					(reference "#PWR012")
 					(unit 1)
 				)
@@
 		(dnp no)
 		(fields_autoplaced yes)
-		(property "Reference" "C3"
+		(property "Reference" "C4"
 			(at 161.29 97.7899 0)
 			(effects
@@
 			)
 		)
-		(property "Footprint" "Capacitor_SMD:C_0805_2012Metric_Pad1.18x1.45mm_HandSolder"
+		(property "Footprint" "Capacitor_SMD:C_0603_1608Metric"
 			(at 158.4452 102.87 0)
 			(effects
@@
 			(project "avionics"
 				(path "/5552e11b-fce5-44fd-aeb8-61bf7d07571f/67ffb272-e6d8-49a0-b0ad-d980ce69be53"
-					(reference "C3")
-					(unit 1)
-				)
+					(reference "C4")
+					(unit 1)
+				)

Commit message: hw: order pcb
Parts:
- removed U3: BMP280, Package_LGA:Bosch_LGA-8_2x2.5mm_P0.65mm_ClockwisePinNumbering, symbol Sensor_Pressure:BMP280
- added U3: BME280, Package_LGA:Bosch_LGA-8_2.5x2.5mm_P0.65mm_ClockwisePinNumbering, symbol Sensor:BME280
- C4, C5: DigiKey Part Number (none) -> 399-C0603C104K5RACTUCT-ND
Connections:
- net +3.3V: now also U3.2 (CSB), U3.6 (VDDIO), U3.8 (VDD)
- net GND: now also U3.1 (GND), U3.5 (SDO), U3.7 (GND)
- net SCL: now also U3.4 (SCK)
- net SDA: now also U3.3 (SDI)
