File: avionics/imu.kicad_sch (KiCad schematic)
At the start: 10 parts, among them U2 BMI088

Commit message: created pcb, nearly done with traces, finalising for ordering soon
Parts:
- U2: footprint Package_LGA:Bosch_LGA-16_4.5x3mm_P0.5mm_LayoutBorder7x1y_ClockwisePinNumbering -> BMI088:PQFN50P450X300X100-16N
Changed lines of the file:
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@@
 			)
 		)
-		(property "Footprint" "Package_LGA:Bosch_LGA-16_4.5x3mm_P0.5mm_LayoutBorder7x1y_ClockwisePinNumbering"
+		(property "Footprint" "BMI088:PQFN50P450X300X100-16N"
 			(at 127 96.52 0)
 			(effects

Commit message: hw: make board smaller, misc hotfixes
Parts:
- removed TP10: TP_INT_GYR, TestPoint:TestPoint_Pad_D1.5mm, symbol Connector:TestPoint
- removed TP4: TP_MISO, TestPoint:TestPoint_Pad_D1.5mm, symbol Connector:TestPoint
- removed TP5: TP_MOSI, TestPoint:TestPoint_Pad_D1.5mm, symbol Connector:TestPoint
- removed TP6: TP_SCK, TestPoint:TestPoint_Pad_D1.5mm, symbol Connector:TestPoint
- removed TP7: TP_CS_GYR, TestPoint:TestPoint_Pad_D1.5mm, symbol Connector:TestPoint
- removed TP8: TP_CS_ACC, TestPoint:TestPoint_Pad_D1.5mm, symbol Connector:TestPoint
- removed TP9: TP_INT_ACC, TestPoint:TestPoint_Pad_D1.5mm, symbol Connector:TestPoint
- C2: renamed from C1; footprint Capacitor_SMD:C_0805_2012Metric_Pad1.18x1.45mm_HandSolder -> Capacitor_SMD:C_0603_1608Metric
- C3: renamed from C2; footprint Capacitor_SMD:C_0805_2012Metric_Pad1.18x1.45mm_HandSolder -> Capacitor_SMD:C_0603_1608Metric
- U2: footprint BMI088:PQFN50P450X300X100-16N -> libraries:PQFN50P450X300X100-16N

Commit message: hw: order pcb
Parts:
- removed U2: BMI088, libraries:PQFN50P450X300X100-16N, symbol Sensor_Motion:BMI088
- added R11: 100k, Resistor_SMD:R_0603_1608Metric, symbol Device:R
- added U2: ISM330DHCX, Package_LGA:LGA-14_3x2.5mm_P0.5mm_LayoutBorder3x4y, symbol Sensor_Motion:ISM330DHCX
- C2, C3: DigiKey Part Number (none) -> 399-C0603C104K5RACTUCT-ND
Connections:
- net +3.3V: now also C3.2, U2.5 (VDDIO), U2.8 (VDD); no longer C3.1
- net GND: now also C3.1, R11.2, U2.2 (SDx), U2.3 (SCx), U2.6 (GND), U2.7 (GND); no longer C3.2
- net INT_ACC: now also U2.4 (INT1)
- net INT_GYR: now also U2.9 (INT2)
- net MISO: now also U2.1 (SDO/SA0)
- net MOSI: now also U2.14 (SDA)
- net SCK: now also U2.13 (SCL)
- new net CS: R11.1, U2.12 (CS)
