File: avionics/psu.kicad_sch (KiCad schematic)
At the start: 27 parts, among them J1 BAT Balancing leads, J2 BAT, U5 TPS548B23VANR

Commit message: created pcb, nearly done with traces, finalising for ordering soon
Parts:
- removed D1: SS24, Diode_SMD:D_SMA, symbol Diode:SS24
- added Q2: AO3401A, Package_TO_SOT_SMD:SOT-23, symbol Transistor_FET:AO3401A
- added R14: 47k, Resistor_SMD:R_0805_2012Metric_Pad1.20x1.40mm_HandSolder, symbol Device:R
Connections:
- net +BATT: now also Q2.3 (D)
- net GND: now also R14.2
- net at C14.1, F1.2: now also Q2.2 (S)
- new net: Q2.1 (G), R14.1
Other:
- moved on the sheet: C14, F1, J2

Commit message: hw: make board smaller, misc hotfixes
Parts:
- removed Q2: AO3401A, Package_TO_SOT_SMD:SOT-23, symbol Transistor_FET:AO3401A
- removed TP14: TP_5V, TestPoint:TestPoint_Pad_D1.5mm, symbol Connector:TestPoint
- added Q1: RF4C050AP, libraries:TRANS_RF4C_ROM, symbol custom:RF4C050AP
- C10: renamed from C9; footprint Capacitor_SMD:C_0805_2012Metric_Pad1.18x1.45mm_HandSolder -> Capacitor_SMD:C_0603_1608Metric
- C11: renamed from C10; footprint Capacitor_SMD:C_0805_2012Metric_Pad1.18x1.45mm_HandSolder -> Capacitor_SMD:C_0603_1608Metric
- C12: renamed from C11; footprint Capacitor_SMD:C_0805_2012Metric_Pad1.18x1.45mm_HandSolder -> Capacitor_SMD:C_0603_1608Metric
- C13: renamed from C12; footprint Capacitor_SMD:C_0805_2012Metric_Pad1.18x1.45mm_HandSolder -> Capacitor_SMD:C_0603_1608Metric
- C14: renamed from C13; footprint Capacitor_SMD:C_0805_2012Metric_Pad1.18x1.45mm_HandSolder -> Capacitor_SMD:C_0603_1608Metric
- C15: renamed from C14; footprint Capacitor_SMD:C_0805_2012Metric_Pad1.18x1.45mm_HandSolder -> Capacitor_SMD:C_0603_1608Metric
- C16: renamed from C15; footprint Capacitor_SMD:C_0805_2012Metric_Pad1.18x1.45mm_HandSolder -> Capacitor_SMD:C_0603_1608Metric
- C17: renamed from C16; footprint Capacitor_SMD:C_0805_2012Metric_Pad1.18x1.45mm_HandSolder -> Capacitor_SMD:C_0603_1608Metric
- C18: renamed from C17; footprint Capacitor_SMD:C_0805_2012Metric_Pad1.18x1.45mm_HandSolder -> Capacitor_SMD:C_0603_1608Metric
- C9: renamed from C8; footprint Capacitor_SMD:C_0805_2012Metric_Pad1.18x1.45mm_HandSolder -> Capacitor_SMD:C_0603_1608Metric
- F1: value Littelfuse 1812L090 -> Littelfuse 2920L400
- J1: footprint Connector_JST:JST_XH_S3B-XH-A_1x03_P2.50mm_Horizontal -> Connector_JST:JST_XH_B3B-XH-A_1x03_P2.50mm_Vertical
- L1: value 300n -> 300n (SRP1038A-R33M); footprint Inductor_SMD:L_2512_6332Metric_Pad1.52x3.35mm_HandSolder -> Inductor_SMD:L_Bourns_SRP1038C_10.0x10.0mm
- R10: renamed from R14; footprint Resistor_SMD:R_0805_2012Metric_Pad1.20x1.40mm_HandSolder -> Resistor_SMD:R_0603_1608Metric
- R11: renamed from R7; footprint Resistor_SMD:R_0805_2012Metric_Pad1.20x1.40mm_HandSolder -> Resistor_SMD:R_0603_1608Metric
- R12: renamed from R8; footprint Resistor_SMD:R_0805_2012Metric_Pad1.20x1.40mm_HandSolder -> Resistor_SMD:R_0603_1608Metric
- R13: renamed from R9; footprint Resistor_SMD:R_0805_2012Metric_Pad1.20x1.40mm_HandSolder -> Resistor_SMD:R_0603_1608Metric
- R6: renamed from R3; footprint Resistor_SMD:R_0805_2012Metric_Pad1.20x1.40mm_HandSolder -> Resistor_SMD:R_0603_1608Metric
- R7: renamed from R4; footprint Resistor_SMD:R_0805_2012Metric_Pad1.20x1.40mm_HandSolder -> Resistor_SMD:R_0603_1608Metric
- R8: renamed from R5; footprint Resistor_SMD:R_0805_2012Metric_Pad1.20x1.40mm_HandSolder -> Resistor_SMD:R_0603_1608Metric
- R9: renamed from R6; footprint Resistor_SMD:R_0805_2012Metric_Pad1.20x1.40mm_HandSolder -> Resistor_SMD:R_0603_1608Metric
Connections:
- net +BATT: now also Q1.1, Q1.2, Q1.5, Q1.6, Q1.7
- net at R10.1: now also Q1.3
- net at C15.1, F1.2: now also Q1.4, Q1.8
Other:
- moved on the sheet: C15, F1, J2

Commit message: hw: order pcb
Parts:
- removed C10: 100n, Capacitor_SMD:C_0603_1608Metric, symbol Device:C
- removed J1: BAT Balancing leads, Connector_JST:JST_XH_B3B-XH-A_1x03_P2.50mm_Vertical, symbol Connector:Conn_01x03_Pin
- removed R6: 10k, Resistor_SMD:R_0603_1608Metric, symbol Device:R
- removed R7: 25k, Resistor_SMD:R_0603_1608Metric, symbol Device:R
- removed R8: 56k, Resistor_SMD:R_0603_1608Metric, symbol Device:R
- removed R9: 33k, Resistor_SMD:R_0603_1608Metric, symbol Device:R
- removed TP12: TP_VBAT_0, TestPoint:TestPoint_Pad_D1.5mm, symbol Connector:TestPoint
- removed TP13: TP_VBAT_1, TestPoint:TestPoint_Pad_D1.5mm, symbol Connector:TestPoint
- added D1: SMF10A, Diode_SMD:D_SMF, symbol Diode:SMF10A
- added R12: 56k, Resistor_SMD:R_0603_1608Metric, symbol Device:R
- added R13: 33k, Resistor_SMD:R_0603_1608Metric, symbol Device:R
- C10: renamed from C11; footprint Capacitor_SMD:C_0603_1608Metric -> Capacitor_SMD:C_1210_3225Metric; DigiKey Part Number (none) -> 1276-1101-1-ND; Mouser Part Number (none) -> 187-CL10A226MP8NUNE
- C11: renamed from C12; footprint Capacitor_SMD:C_0603_1608Metric -> Capacitor_SMD:C_1210_3225Metric; DigiKey Part Number (none) -> 1276-1101-1-ND; Mouser Part Number (none) -> 187-CL10A226MP8NUNE
- C12: renamed from C13; DigiKey Part Number (none) -> 587-2400-1-ND; Mouser Part Number (none) -> 80-C0603C391K3G
- C13: renamed from C14; DigiKey Part Number (none) -> 587-2400-1-ND; Mouser Part Number (none) -> 80-C0603C391K3G
- C14: renamed from C15; DigiKey Part Number (none) -> 399-C0603C104K5RACTUCT-ND; Mouser Part Number (none) -> 603-CC603KRX5R9BB104
- C15: renamed from C16; DigiKey Part Number (none) -> 587-2400-1-ND; Mouser Part Number (none) -> 80-C0603C391K3G
- C16: renamed from C17; DigiKey Part Number (none) -> 399-C0603C104K5RACTUCT-ND; Mouser Part Number (none) -> 603-CC603KRX5R9BB104
- C17: renamed from C18; footprint Capacitor_SMD:C_0603_1608Metric -> Capacitor_SMD:C_1210_3225Metric; DigiKey Part Number (none) -> 490-8354-1-ND; Mouser Part Number (none) -> 81-GRM188R60J476ME5D
- C9: DigiKey Part Number (none) -> 399-C0603C104K5RACTUCT-ND
- F1: footprint Fuse:Fuse_1812_4532Metric_Pad1.30x3.40mm_HandSolder -> Fuse:Fuse_2920_7451Metric; DigiKey Part Number (none) -> F8136CT-ND; Mouser Part Number (none) -> 576-2920L400/15MR
- J1: renamed from J2; value BAT -> XT60M; footprint Connector_Molex:Molex_Mini-Fit_Jr_5566-02A_2x01_P4.20mm_Vertical -> Connector_AMASS:AMASS_XT60-M_1x02_P7.20mm_Vertical; DigiKey Part Number (none) -> 1738-1437-ND; LCSC Part Number (none) -> C98733
- L1: value 300n (SRP1038A-R33M) -> 300n; DigiKey Part Number (none) -> 118-SRP1038A-R33MCT-ND; Manufacturer_Part_Number (none) -> SRP1038A-R33M; Mouser Part Number (none) -> 652-SRP1038A-R33M
- Q1: DigiKey Part Number (none) -> RF4C050APCT-ND; Mouser Part Number (none) -> 755-RF4C050APTR
- R14: renamed from R10; DigiKey Part Number (none) -> 311-47.0KHRCT-ND; Mouser Part Number (none) -> 594-MCT06030D4702BP5
- R15: renamed from R11; DigiKey Part Number (none) -> P37.4HCT-ND; Mouser Part Number (none) -> 71-CRCW0603-37.4K-E3
- R16: renamed from R12; DigiKey Part Number (none) -> 311-10.0KHRCT-ND; Mouser Part Number (none) -> 594-MCT06030C1022FP5
- R17: renamed from R13; DigiKey Part Number (none) -> 311-10.0KHRCT-ND; Mouser Part Number (none) -> 594-MCT06030C1022FP5
- TP2: renamed from TP15; now left out of the parts list
- U5: DigiKey Part Number (none) -> TPS548B23VANR; Mouser Part Number (none) -> 595-TPS548B23VANR
Connections:
- net +BATT: now also R12.1
- net GND: now also D1.2 (A2), R13.2
- net BAT_CONN+: now reaches F1.1, J1.2 (Pin_2)
- net BAT_CONN+: now also D1.1 (A1)
- net BAT_CELL_0 renamed BAT_VOLTAGE
- net BAT_VOLTAGE: now also R12.2, R13.1
Other:
- note added: "Battery reverse-polarity, overcurrent, ESD protection"
- note removed: "Battery reverse-polarity and overcurrent protection"
- note removed: "Battery voltage sensing"
- moved on the sheet: C14, F1, J1
